File: flowerpower/GPIO.sch (KiCad schematic (older format))
At the start: 3 parts, among them J10 GPIO, J9 Power select

Commit message: beginning layout
Changed lines of the file:
@@
 $Descr A4 11693 8268
 encoding utf-8
-Sheet 3 11
+Sheet 5 11
 Title ""
 Date ""
@@
 AR Path="/5F95F7DC/5F95761F" Ref="J12"  Part="1"
 AR Path="/5F965BCA/5F95761F" Ref="J14"  Part="1"
-F 0 "J10" H 6318 3325 50  0000 C CNN
+F 0 "J14" H 6318 3325 50  0000 C CNN
 F 1 "GPIO" H 6318 3416 50  0000 C CNN
 F 2 "Pin_Headers:Pin_Header_Straight_1x03" H 6400 3650 50  0001 C CNN
@@
 AR Path="/5F95F7DC/5F957625" Ref="J11"  Part="1"
 AR Path="/5F965BCA/5F957625" Ref="J13"  Part="1"
-F 0 "J9" H 4818 3967 50  0000 C CNN
+F 0 "J13" H 4818 3967 50  0000 C CNN
 F 1 "Power select" H 4818 3876 50  0000 C CNN
 F 2 "Pin_Headers:Pin_Header_Straight_1x03" H 4900 3650 50  0001 C CNN
@@
 AR Path="/5F95F7DC/5F96CA2C" Ref="C15"  Part="1"
 AR Path="/5F965BCA/5F96CA2C" Ref="C16"  Part="1"
-F 0 "C14" H 5865 3846 50  0000 L CNN
+F 0 "C16" H 5865 3846 50  0000 L CNN
 F 1 "100N" H 5865 3755 50  0000 L CNN
 F 2 "Capacitors_SMD:C_0603" H 5788 3650 50  0001 C CNN
