File: flowerpower/flowerpower.kicad_pcb (KiCad board)
At the start: 2 copper layers, 133 parts, among them J1 Power In, J10 GPIO, J11 Power select, J12 GPIO, J13 Power select, J14 GPIO, J15 Switched, J16 Switched, J17 Water sense, J18 Motor, J19 Water sense, J2 ESP_DEBUG, J20 Motor, J21 Water sense, J22 Motor, J23 Water sense, J24 Motor, J3 ESP8266, J4 USB_B_Micro, J5 Water E-stop, J6 SWD, J7 Water sense, J8 Motor, J9 Power select, K1 G5Q-1A, K2 G5Q-1A, Q1 RK7002BM, Q2 RK7002BM, SW1 BOOT, U1 LM2576HVS-5, U2 NCP1117-3.3_SOT223, U3 74HC14, U4 STM32F051C6Tx, U5 TB6559, U6 TB6559, U7 TB6559, U8 TB6559, U9 TB6559, Y1 32.768K

Commit message: tweaking layout
Parts:
- added REF**: MountingHole_3.7mm, Mounting_Holes:MountingHole_3.7mm, F.Cu at (180.3, 54.0)
- added REF**: MountingHole_3.7mm, Mounting_Holes:MountingHole_3.7mm, F.Cu at (220.3, 108.6)
- C3, C4, C5: footprint Capacitors_SMD:C_0603 -> Capacitors_SMD:C_0805
- moved C3 116.4 mm to (167.6, 94.6)
- moved D2 96.6 mm to (142.2, 61.0)
- moved R1 91.3 mm to (142.2, 64.1), turned to 0 degrees
- moved C7 82.7 mm to (103.4, 80.6), turned to 180 degrees
- moved D3 80.8 mm to (120.7, 61.6)
- moved Y1 80.4 mm to (105.4, 87.6), turned to 270 degrees
- moved C9 79.9 mm to (120.5, 94.6), turned to 180 degrees
- moved C5 73.0 mm to (128.3, 77.2), turned to 90 degrees
- moved C29 71.9 mm to (135.9, 91.4), turned to 180 degrees
- moved R5 69.2 mm to (119.5, 76.2)
- moved R2 56.7 mm to (120.7, 65.4)
- moved C4 56.0 mm to (128.3, 72.4), turned to 270 degrees
- moved TP1 55.3 mm to (97.8, 53.3)
- moved C10 49.9 mm to (112.9, 80.6)
- moved J2 48.9 mm to (106.7, 61.6), turned to 90 degrees
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Routing:
- net Net-(D10-Pad2): track 11.7 -> 21.2 mm
- net Net-(D12-Pad2): track 11.7 -> 21.2 mm
- net Net-(J16-Pad1): track 14.7 -> 23.8 mm
- net Net-(J15-Pad1): track 14.7 -> 23.8 mm
- net Net-(F1-Pad2): track 21.8 -> 16.0 mm
- net Net-(F2-Pad2): track 21.8 -> 16.0 mm
- net Net-(F2-Pad1): track 9.10 -> 13.7 mm
- net Net-(F1-Pad1): track 9.10 -> 13.7 mm
- net +5V: track 14.2 -> 16.5 mm

Commit message: finish layout
Parts:
- added C31: 100n, Capacitors_SMD:C_0603, F.Cu at (109.9, 88.3)
- added C32: 100n, Capacitors_SMD:C_0603, F.Cu at (122.6, 80.6)
- U4: value STM32F051C6Tx -> STM32F041C6Tx
- moved C24 24.1 mm to (157.5, 113.0)
- moved C25 24.1 mm to (157.5, 119.4)
- moved C27 24.1 mm to (181.6, 113.0)
- moved C28 24.1 mm to (181.6, 119.4)
- moved U6 24.1 mm to (118.1, 115.6)
- moved U7 24.1 mm to (142.2, 115.6)
- moved C17 24.1 mm to (128.3, 120.7), turned to 0 degrees
- moved C18 24.1 mm to (109.2, 113.0)
- moved C19 24.1 mm to (109.2, 119.4)
- moved C20 24.1 mm to (152.4, 120.7)
- moved C21 24.1 mm to (133.3, 113.0)
- moved C22 24.1 mm to (133.3, 119.4)
- moved C23 24.1 mm to (176.5, 120.7), turned to 180 degrees
- moved C26 24.1 mm to (200.7, 120.7)
- moved D14 24.1 mm to (128.3, 127.0)
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Connections:
- C1 pad 1: +VDC -> VDC
- C30 pad 1: +VDC -> VDC
- J1 pad 1: +VDC -> VDC
- J4 pad 6: GND -> Net-(J4-Pad6)
- U1 pad 1: +VDC -> VDC
- U4 pad 10: Net-(U4-Pad10) -> /P1A
- U4 pad 11: Net-(U4-Pad11) -> /P1B
- U4 pad 12: Net-(U4-Pad12) -> /P2A
- U4 pad 13: Net-(U4-Pad13) -> /P2B
- U4 pad 16: Net-(U4-Pad16) -> /P3A
- U4 pad 17: Net-(U4-Pad17) -> /P3B
- U4 pad 18: Net-(U4-Pad18) -> /P4A
- U4 pad 19: Net-(U4-Pad19) -> /GPIO1
- U4 pad 20: Net-(U4-Pad20) -> /P1W
- U4 pad 21: Net-(U4-Pad21) -> /P2W
- U4 pad 22: Net-(U4-Pad22) -> /P3W
- U4 pad 25: Net-(U4-Pad25) -> /P4W
- U4 pad 26: Net-(U4-Pad26) -> /P4B
- U4 pad 27: Net-(U4-Pad27) -> /P5A
- U4 pad 28: Net-(U4-Pad28) -> /P5B
- U4 pad 29: Net-(U4-Pad29) -> /P5W
- U4 pad 35: Net-(U4-Pad35) -> GND
- U4 pad 36: Net-(U4-Pad36) -> +3V3
- U4 pad 45: Net-(U4-Pad45) -> /GPIO2
- U4 pad 46: Net-(U4-Pad46) -> /GPIO3
Routing:
- net GND: track 0.00 -> 356.2 mm, vias 0 -> 99
- net (no net): track 300.5 -> 0.00 mm, vias 8 -> 0
- net VDC: track 22.4 -> 261.1 mm, vias 0 -> 19
- net +5V: track 16.5 -> 232.4 mm, vias 0 -> 4
- net +3V3: track 0.00 -> 104.2 mm, vias 0 -> 20
- net /P5W: track 0.00 -> 103.5 mm, vias 0 -> 2
- net /P5B: track 0.00 -> 102.8 mm, vias 0 -> 2
- net /WATER_ESTOP: track 0.00 -> 97.5 mm, vias 0 -> 2
- net Net-(C6-Pad1): track 16.5 -> 110.7 mm, vias 0 -> 2
- net /P5A: track 0.00 -> 90.9 mm, vias 0 -> 2
- net /P4B: track 0.00 -> 77.1 mm, vias 0 -> 2
- net /P4A: track 0.00 -> 74.6 mm, vias 0 -> 2
- net /Pot 4/INV_IN: track 0.00 -> 67.3 mm
- net /Pot 5/INV_IN: track 28.5 -> 95.3 mm
- net /P4W: track 13.3 -> 78.1 mm, vias 0 -> 2
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- added copper zone on F.Cu, net +3V3
- added copper zone on B.Cu, net GND

Commit message: silkscreen
Parts:
- moved REF** 0.64 mm to (141.6, 54.0)
- moved REF** 0.64 mm to (220.3, 109.2)
- moved REF** 0.63 mm to (179.7, 54.0)
Routing:
- net +3V3: track 104.2 -> 107.4 mm
Other:
- board outline added: 142.2 x 89.5 mm
- rule trace_min: 0.2 -> 0
- board text added: "+"
- board text added: "-"
- board text added: "1"
- board text added: "10A Max"
- board text added: "2"
- board text added: "3"
- board text added: "3.3V"
- board text added: "4"
- board text added: "5"
- board text added: "5V"
- board text added: "7-24V"
- board text added: "DC Power"
- board text added: "Drain"
- board text added: "ESP"
- board text added: "ESP8266"
- board text added: "Flood"
- board text added: "Flower Power"
- board text added: "Full"
- board text added: "GPIO"
- board text added: "M3.5 or #6"
- board text added: "MCU Power"
- board text added: "Overflow"
- board text added: "Pump"
- board text added: "RX"
- board text added: "Relay"
- board text added: "SWD"
- board text added: "Sense"
- board text added: "TX"
- board text added: "by Eric Van Albert"
- board text added: "rev 1"

Commit message: Final tweaks
Parts:
- removed the REF** at (87.0, 54.0)
- removed the REF** at (220.3, 54.0)
- added D26: YELLOW, LEDs:LED_0603, F.Cu at (109.2, 62.2)
- added R28: 470R, Resistors_SMD:R_0603, F.Cu at (120.7, 73.7)
- added REF**: MountingHole_3.7mm, Mounting_Holes:MountingHole_3.7mm, F.Cu at (87.0, 54.6)
- added REF**: MountingHole_3.7mm, Mounting_Holes:MountingHole_3.7mm, F.Cu at (220.3, 54.6)
- J15, J16: footprint Terminal_Blocks:TerminalBlock_Pheonix_MPT-2.54mm_2pol -> Terminal_Blocks:TerminalBlock_Pheonix_PT-3.5mm_2pol
- moved J3 7.62 mm to (114.3, 76.8), turned to 270 degrees
- moved R5 5.21 mm to (120.7, 69.8)
- moved J15 2.01 mm to (217.8, 66.7)
- moved J16 2.01 mm to (217.8, 94.6)
- moved D10 1.27 mm to (184.2, 71.1)
- moved Q1 1.27 mm to (179.1, 71.1)
- moved U2 1.27 mm to (133.3, 82.5)
- moved SW1 1.27 mm to (109.2, 55.9)
- moved D11 1.27 mm to (184.2, 64.8)
- moved D12 1.27 mm to (184.2, 99.1)
- moved D13 1.27 mm to (184.2, 92.7)
- moved D2 1.27 mm to (142.2, 62.2)
- moved F1 1.27 mm to (207.0, 64.8)
- moved F2 1.27 mm to (207.0, 92.7)
- moved K1 1.27 mm to (198.1, 73.7)
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Connections:
- U4 pad 40: Net-(U4-Pad40) -> /HEARTBEAT
Routing:
- net +5V: track 232.4 -> 216.2 mm, vias 4 -> 6
- net Net-(D26-Pad2): track 0.00 -> 15.9 mm
- net /HEARTBEAT: track 0.00 -> 11.0 mm, vias 0 -> 2
- net +3V3: track 107.4 -> 101.8 mm, vias 20 -> 13
- net /P1A: track 48.6 -> 53.7 mm, vias 0 -> 2
- net /ESP_RESET: track 12.4 -> 15.8 mm
- net /SWCLK: track 19.9 -> 22.3 mm
- net /ESP_TX: track 36.0 -> 38.0 mm, vias 0 -> 1
- net /OSC32_OUT: track 15.5 -> 13.7 mm
- net GND: track 356.2 -> 357.8 mm, vias 99 -> 100
- net /P4A: track 74.6 -> 75.7 mm
- net /P1B: track 43.6 -> 44.6 mm, vias 0 -> 2
- net /ESP_RX: track 34.5 -> 33.5 mm
- net /Pot 3/INV_IN: track 43.1 -> 43.9 mm, vias 0 -> 2
- net Net-(D1-Pad1): track 22.2 -> 21.6 mm
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Other:
- board size 142.2 x 89.5 mm -> 142.2 x 88.9 mm
- board text added: "Boot"
- board text added: "Heartbeat"
