File: flowerpower/flowerpower.sch (KiCad schematic (older format))
At the start: 36 parts, among them J1 Power In, J2 ESP_DEBUG, J3 ESP8266, J4 USB_B_Micro, J5 Water E-stop, J6 SWD, SW1 BOOT, U1 LM2576HVS-5, U2 NCP1117-3.3_SOT223, U3 74HC14, U4 STM32F051C6Tx, Y1 32.768K

Commit message: beginning layout
Parts:
- removed J1: Power In, symbol Connector:Barrel_Jack_MountingPin
- added C30: 10U, Capacitors_SMD:C_1206, symbol Device:C
- added J1: Power In, Connect:BARREL_JACK, symbol Connector:Barrel_Jack_Switch
- C1: value CP -> 100U; footprint (none) -> Capacitors_SMD:c_elec_10x10
- C2: footprint (none) -> Capacitors_SMD:c_elec_10x10
- L1: footprint (none) -> flowerpower:toroid_14.2_32.5dia
- U1: footprint Package_TO_SOT_SMD:TO-263-5_TabPin3 -> TO_SOT_Packages_SMD:TO-263-5Lead
- U2: footprint Package_TO_SOT_SMD:SOT-223-3_TabPin2 -> TO_SOT_Packages_SMD:SOT-223
- U3: footprint (none) -> Housings_SOIC:SOIC-14_3.9x8.7mm_Pitch1.27mm
- U4: footprint Package_QFP:LQFP-48_7x7mm_P0.5mm -> Housings_QFP:LQFP-48_7x7mm_Pitch0.5mm
- Y1: footprint (none) -> flowerpower:SOJ-4
Connections:
- net +VDC: now also C30.1, J1.1
- net GND: now also C30.2, J1.2, J1.3
Other:
- moved on the sheet: C1
Changed lines of the file:
@@
 F 0 "U4" H 2800 3100 50  0000 C CNN
 F 1 "STM32F051C6Tx" H 3050 3000 50  0000 C CNN
-F 2 "Package_QFP:LQFP-48_7x7mm_P0.5mm" H 2950 3250 50  0001 R CNN
+F 2 "Housings_QFP:LQFP-48_7x7mm_Pitch0.5mm" H 2950 3250 50  0001 R CNN
 F 3 "http://www.st.com/st-web-ui/static/active/en/resource/technical/document/datasheet/DM00039193.pdf" H 3450 4750 50  0001 C CNN
 	1    3450 4750
@@
 F 0 "U1" H 2450 1267 50  0000 C CNN
 F 1 "LM2576HVS-5" H 2450 1176 50  0000 C CNN
-F 2 "Package_TO_SOT_SMD:TO-263-5_TabPin3" H 2450 650 50  0001 L CIN
+F 2 "TO_SOT_Packages_SMD:TO-263-5Lead" H 2450 650 50  0001 L CIN
 F 3 "http://www.ti.com/lit/ds/symlink/lm2576.pdf" H 2450 900 50  0001 C CNN
 	1    2450 900
@@
 F 0 "L1" V 3250 1000 50  0000 C CNN
 F 1 "330U" V 3399 1000 50  0000 C CNN
-F 2 "" H 3300 1000 50  0001 C CNN
+F 2 "flowerpower:toroid_14.2_32.5dia" H 3300 1000 50  0001 C CNN
 F 3 "~" H 3300 1000 50  0001 C CNN
 	1    3300 1000
@@
 L power:GND #PWR07
 U 1 1 5F7F489D
-P 1600 1100
-F 0 "#PWR07" H 1600 850 50  0001 C CNN
-F 1 "GND" H 1605 927 50  0000 C CNN
-F 2 "" H 1600 1100 50  0001 C CNN
-F 3 "" H 1600 1100 50  0001 C CNN
-	1    1600 1100
-	1    0    0    -1
-$EndComp
-$Comp
-L Connector:Barrel_Jack_MountingPin J1
-U 1 1 5F7F52E4
-P 900 900
-F 0 "J1" H 957 1217 50  0000 C CNN
-F 1 "Power In" H 957 1126 50  0000 C CNN
-F 2 "" H 950 860 50  0001 C CNN
-F 3 "~" H 950 860 50  0001 C CNN
-	1    900  900
-	1    0    0    -1
-$EndComp
-Wire Wire Line
-	1200 1000 1200 1200
-Wire Wire Line
-	1200 1200 900  1200
-Wire Wire Line
-	1200 1200 1200 1300
-Connection ~ 1200 1200
+P 1400 1100
+F 0 "#PWR07" H 1400 850 50  0001 C CNN
+F 1 "GND" H 1405 927 50  0000 C CNN
+F 2 "" H 1400 1100 50  0001 C CNN
+F 3 "" H 1400 1100 50  0001 C CNN
+	1    1400 1100
+	1    0    0    -1
+$EndComp
 $Comp
 L power:GND #PWR010
@@
 L Device:CP C1
 U 1 1 5F805496
-P 1600 950
-F 0 "C1" H 1718 996 50  0000 L CNN
-F 1 "CP" H 1718 905 50  0000 L CNN
-F 2 "" H 1638 800 50  0001 C CNN
-F 3 "~" H 1600 950 50  0001 C CNN
-	1    1600 950
-	1    0    0    -1
-$EndComp
-Wire Wire Line
-	1200 800  1600 800
+P 1400 950
+F 0 "C1" H 1300 1300 50  0000 L CNN
+F 1 "100U" H 1300 1200 50  0000 L CNN
+F 2 "Capacitors_SMD:c_elec_10x10" H 1438 800 50  0001 C CNN
+F 3 "~" H 1400 950 50  0001 C CNN
+	1    1400 950
+	1    0    0    -1
+$EndComp
+Wire Wire Line
+	1200 800  1400 800
 Connection ~ 1600 800
 Wire Wire Line
-	1600 800  1950 800
+	1600 800  1750 800
 $Comp
 L Device:CP C2
@@
 F 0 "C2" H 3668 1296 50  0000 L CNN
 F 1 "330U" H 3668 1205 50  0000 L CNN
-F 2 "" H 3588 1100 50  0001 C CNN
+F 2 "Capacitors_SMD:c_elec_10x10" H 3588 1100 50  0001 C CNN
 F 3 "~" H 3550 1250 50  0001 C CNN
 	1    3550 1250
@@
 F 0 "U2" H 4650 2342 50  0000 C CNN
 F 1 "NCP1117-3.3_SOT223" H 4650 2251 50  0000 C CNN
-F 2 "Package_TO_SOT_SMD:SOT-223-3_TabPin2" H 4650 2300 50  0001 C CNN
+F 2 "TO_SOT_Packages_SMD:SOT-223" H 4650 2300 50  0001 C CNN
 F 3 "http://www.onsemi.com/pub_link/Collateral/NCP1117-D.PDF" H 4750 1850 50  0001 C CNN
 	1    4650 2100
@@
 F 0 "Y1" H 1250 4868 50  0000 C CNN
 F 1 "32.768K" H 1250 4777 50  0000 C CNN
-F 2 "" H 1250 4600 50  0001 C CNN
+F 2 "flowerpower:SOJ-4" H 1250 4600 50  0001 C CNN
 F 3 "~" H 1250 4600 50  0001 C CNN
 	1    1250 4600
@@
 F 0 "U3" H 7550 2517 50  0000 C CNN
 F 1 "74HC14" H 7550 2426 50  0000 C CNN
-F 2 "" H 7550 2200 50  0001 C CNN
+F 2 "Housings_SOIC:SOIC-14_3.9x8.7mm_Pitch1.27mm" H 7550 2200 50  0001 C CNN
 F 3 "http://www.ti.com/lit/gpn/sn74HC14" H 7550 2200 50  0001 C CNN
 	1    7550 2200
@@
 F 0 "U3" H 6750 3517 50  0000 C CNN
 F 1 "74HC14" H 6750 3426 50  0000 C CNN
-F 2 "" H 6750 3200 50  0001 C CNN
+F 2 "Housings_SOIC:SOIC-14_3.9x8.7mm_Pitch1.27mm" H 6750 3200 50  0001 C CNN
 F 3 "http://www.ti.com/lit/gpn/sn74HC14" H 6750 3200 50  0001 C CNN
 	2    6750 3200
@@
 F 0 "U3" H 6750 4267 50  0000 C CNN
 F 1 "74HC14" H 6750 4176 50  0000 C CNN
-F 2 "" H 6750 3950 50  0001 C CNN
+F 2 "Housings_SOIC:SOIC-14_3.9x8.7mm_Pitch1.27mm" H 6750 3950 50  0001 C CNN
 F 3 "http://www.ti.com/lit/gpn/sn74HC14" H 6750 3950 50  0001 C CNN
 	3    6750 3950
@@
 F 0 "U3" H 6750 5017 50  0000 C CNN
 F 1 "74HC14" H 6750 4926 50  0000 C CNN
-F 2 "" H 6750 4700 50  0001 C CNN
+F 2 "Housings_SOIC:SOIC-14_3.9x8.7mm_Pitch1.27mm" H 6750 4700 50  0001 C CNN
 F 3 "http://www.ti.com/lit/gpn/sn74HC14" H 6750 4700 50  0001 C CNN
 	4    6750 4700
@@
 F 0 "U3" H 6750 5767 50  0000 C CNN
 F 1 "74HC14" H 6750 5676 50  0000 C CNN
-F 2 "" H 6750 5450 50  0001 C CNN
+F 2 "Housings_SOIC:SOIC-14_3.9x8.7mm_Pitch1.27mm" H 6750 5450 50  0001 C CNN
 F 3 "http://www.ti.com/lit/gpn/sn74HC14" H 6750 5450 50  0001 C CNN
 	5    6750 5450
@@
 F 0 "U3" H 6750 6517 50  0000 C CNN
 F 1 "74HC14" H 6750 6426 50  0000 C CNN
-F 2 "" H 6750 6200 50  0001 C CNN
+F 2 "Housings_SOIC:SOIC-14_3.9x8.7mm_Pitch1.27mm" H 6750 6200 50  0001 C CNN
 F 3 "http://www.ti.com/lit/gpn/sn74HC14" H 6750 6200 50  0001 C CNN
 	6    6750 6200
@@
 F 0 "U3" H 7700 5000 50  0000 C CNN
 F 1 "74HC14" V 7650 5400 50  0000 C CNN
-F 2 "" H 7900 5400 50  0001 C CNN
+F 2 "Housings_SOIC:SOIC-14_3.9x8.7mm_Pitch1.27mm" H 7900 5400 50  0001 C CNN
 F 3 "http://www.ti.com/lit/gpn/sn74HC14" H 7900 5400 50  0001 C CNN
 	7    7900 5400
@@
 	1    0    0    -1
 $EndComp
+Connection ~ 1400 800
+Wire Wire Line
+	1400 800  1600 800
+$Comp
+L Device:C C30
+U 1 1 5F776BE6
+P 1750 950
+F 0 "C30" H 1750 1300 50  0000 L CNN
+F 1 "10U" H 1750 1200 50  0000 L CNN
+F 2 "Capacitors_SMD:C_1206" H 1788 800 50  0001 C CNN
+F 3 "~" H 1750 950 50  0001 C CNN
+	1    1750 950
+	1    0    0    -1
+$EndComp
+Connection ~ 1750 800
+Wire Wire Line
+	1750 800  1950 800
+$Comp
+L power:GND #PWR0120
+U 1 1 5F777303
+P 1750 1100
+F 0 "#PWR0120" H 1750 850 50  0001 C CNN
+F 1 "GND" H 1755 927 50  0000 C CNN
+F 2 "" H 1750 1100 50  0001 C CNN
+F 3 "" H 1750 1100 50  0001 C CNN
+	1    1750 1100
+	1    0    0    -1
+$EndComp
+$Comp
+L Connector:Barrel_Jack_Switch J1
+U 1 1 5F7B8483
+P 900 900
+F 0 "J1" H 957 1217 50  0000 C CNN
+F 1 "Power In" H 957 1126 50  0000 C CNN
+F 2 "Connect:BARREL_JACK" H 950 860 50  0001 C CNN
+F 3 "~" H 950 860 50  0001 C CNN
+	1    900  900
+	1    0    0    -1
+$EndComp
+Wire Wire Line
+	1200 900  1200 1000
+Connection ~ 1200 1000
+Wire Wire Line
+	1200 1000 1200 1300
 $EndSCHEMATC

Commit message: tweaking layout
Parts:
- C3, C4, C5: footprint Capacitors_SMD:C_0603 -> Capacitors_SMD:C_0805
Changed lines of the file:
@@
 F 0 "C4" H 4015 2296 50  0000 L CNN
 F 1 "2u2" H 4015 2205 50  0000 L CNN
-F 2 "Capacitors_SMD:C_0603" H 3938 2100 50  0001 C CNN
+F 2 "Capacitors_SMD:C_0805" H 3938 2100 50  0001 C CNN
 F 3 "~" H 3900 2250 50  0001 C CNN
 	1    3900 2250
@@
 F 0 "C5" H 5165 2296 50  0000 L CNN
 F 1 "2u2" H 5165 2205 50  0000 L CNN
-F 2 "Capacitors_SMD:C_0603" H 5088 2100 50  0001 C CNN
+F 2 "Capacitors_SMD:C_0805" H 5088 2100 50  0001 C CNN
 F 3 "~" H 5050 2250 50  0001 C CNN
 	1    5050 2250
@@
 F 0 "C3" H 4215 1296 50  0000 L CNN
 F 1 "2u2" H 4215 1205 50  0000 L CNN
-F 2 "Capacitors_SMD:C_0603" H 4138 1100 50  0001 C CNN
+F 2 "Capacitors_SMD:C_0805" H 4138 1100 50  0001 C CNN
 F 3 "~" H 4100 1250 50  0001 C CNN
 	1    4100 1250

Commit message: finish layout
Parts:
- added C31, C32: 100n, Capacitors_SMD:C_0603, symbol Device:C
- U4: value STM32F051C6Tx -> STM32F041C6Tx
Connections:
- net +3V3: now also U4.36 (PF7), C31.1, C32.1
- net GND: now also U4.35 (PF6), C31.2, C32.2; no longer J4.6 (Shield)
- net GPIO1: now also U4.19 (PB1)
- net GPIO2: now also U4.45 (PB8)
- net GPIO3: now also U4.46 (PB9)
- net P1A: now also U4.10 (PA0)
- net P1B: now also U4.11 (PA1)
- net P1W: now also U4.20 (PB2)
- net P2A: now also U4.12 (PA2)
- net P2B: now also U4.13 (PA3)
- net P2W: now also U4.21 (PB10)
- net P3A: now also U4.16 (PA6)
- net P3B: now also U4.17 (PA7)
- net P3W: now also U4.22 (PB11)
- net P4A: now also U4.18 (PB0)
- net P4B: now also U4.26 (PB13)
- net P4W: now also U4.25 (PB12)
- net P5A: now also U4.27 (PB14)
- net P5B: now also U4.28 (PB15)
- net P5W: now also U4.29 (PA8)
- net +VDC renamed VDC
- no-connect marks 4 -> 14
Changed lines of the file:
@@
 Comment4 ""
 $EndDescr
-$Comp
-L MCU_ST_STM32F0:STM32F051C6Tx U4
-U 1 1 5F72889D
-P 3450 4750
-F 0 "U4" H 2800 3100 50  0000 C CNN
-F 1 "STM32F051C6Tx" H 3050 3000 50  0000 C CNN
-F 2 "Housings_QFP:LQFP-48_7x7mm_Pitch0.5mm" H 2950 3250 50  0001 R CNN
-F 3 "http://www.st.com/st-web-ui/static/active/en/resource/technical/document/datasheet/DM00039193.pdf" H 3450 4750 50  0001 C CNN
-	1    3450 4750
-	1    0    0    -1
-$EndComp
 Wire Wire Line
 	3350 6350 3450 6350
@@
 F 3 "" H 3450 6450 50  0001 C CNN
 	1    3450 6450
-	1    0    0    -1
-$EndComp
-$Comp
-L Connector:USB_B_Micro J4
-U 1 1 5BE2379A
-P 2200 2300
-F 0 "J4" H 2255 2767 50  0000 C CNN
-F 1 "USB_B_Micro" H 2255 2676 50  0000 C CNN
-F 2 "Connect:USB_Micro-B" H 2350 2250 50  0001 C CNN
-F 3 "~" H 2350 2250 50  0001 C CNN
-	1    2200 2300
 	1    0    0    -1
 $EndComp
@@
 Text Label 1950 3550 0    50   ~ 0
 BUTTON
-Wire Wire Line
-	2100 2700 2200 2700
 $Comp
 L Device:C C9
@@
 Wire Wire Line
 	4050 5750 4600 5750
-Connection ~ 2200 2700
 Text Label 4600 5750 2    50   ~ 0
 USB_DM
@@
 Wire Wire Line
 	1200 800  1400 800
-Connection ~ 1600 800
-Wire Wire Line
-	1600 800  1750 800
 $Comp
 L Device:CP C2
@@
 F 3 "http://www.onsemi.com/pub_link/Collateral/NCP1117-D.PDF" H 4750 1850 50  0001 C CNN
 	1    4650 2100
-	1    0    0    -1
-$EndComp
-$Comp
-L power:+VDC #PWR01
-U 1 1 5F82049D
-P 1600 800
-F 0 "#PWR01" H 1600 700 50  0001 C CNN
-F 1 "+VDC" H 1600 1075 50  0000 C CNN
-F 2 "" H 1600 800 50  0001 C CNN
-F 3 "" H 1600 800 50  0001 C CNN
-	1    1600 800
 	1    0    0    -1
 $EndComp
@@
 $EndComp
 Connection ~ 1400 800
-Wire Wire Line
-	1400 800  1600 800
 $Comp
 L Device:C C30
@@
 Wire Wire Line
 	1200 1000 1200 1300
+$Comp
+L Device:C C31
+U 1 1 5F99DE7B
+P 4050 7200
+F 0 "C31" H 4165 7246 50  0000 L CNN
+F 1 "100n" H 4165 7155 50  0000 L CNN
+F 2 "Capacitors_SMD:C_0603" H 4088 7050 50  0001 C CNN
+F 3 "~" H 4050 7200 50  0001 C CNN
+	1    4050 7200
+	1    0    0    -1
+$EndComp
+$Comp
+L power:+3V3 #PWR0121
+U 1 1 5F99DE85
+P 4050 7050
+F 0 "#PWR0121" H 4050 6900 50  0001 C CNN
+F 1 "+3V3" H 4065 7223 50  0000 C CNN
+F 2 "" H 4050 7050 50  0001 C CNN
+F 3 "" H 4050 7050 50  0001 C CNN
+	1    4050 7050
+	1    0    0    -1
+$EndComp
+$Comp
+L power:GND #PWR0122
+U 1 1 5F99DE8F
+P 4050 7350
+F 0 "#PWR0122" H 4050 7100 50  0001 C CNN
+F 1 "GND" H 4055 7177 50  0000 C CNN
+F 2 "" H 4050 7350 50  0001 C CNN
+F 3 "" H 4050 7350 50  0001 C CNN
+	1    4050 7350
+	1    0    0    -1
+$EndComp
+$Comp
+L power:+3V3 #PWR0123
+U 1 1 5F9F7CEB
+P 2700 4100
+F 0 "#PWR0123" H 2700 3950 50  0001 C CNN
+F 1 "+3V3" V 2715 4228 50  0000 L CNN
+F 2 "" H 2700 4100 50  0001 C CNN
+F 3 "" H 2700 4100 50  0001 C CNN
+	1    2700 4100
+	0    -1   -1   0
+$EndComp
+$Comp
+L power:GND #PWR0124
+U 1 1 5F9F902F
+P 2700 3900
+F 0 "#PWR0124" H 2700 3650 50  0001 C CNN
+F 1 "GND" H 2705 3727 50  0000 C CNN
+F 2 "" H 2700 3900 50  0001 C CNN
+F 3 "" H 2700 3900 50  0001 C CNN
+	1    2700 3900
+	0    1    1    0
+$EndComp
+Wire Wire Line
+	2850 3950 2750 3950
+Wire Wire Line
+	2750 3950 2750 3900
+Wire Wire Line
+	2750 3900 2700 3900
+Wire Wire Line
+	2700 4100 2750 4100
+Wire Wire Line
+	2750 4100 2750 4050
+Wire Wire Line
+	2750 4050 2850 4050
+$Comp
+L Device:C C32
+U 1 1 5FA08621
+P 4500 7200
+F 0 "C32" H 4615 7246 50  0000 L CNN
+F 1 "100n" H 4615 7155 50  0000 L CNN
+F 2 "Capacitors_SMD:C_0603" H 4538 7050 50  0001 C CNN
+F 3 "~" H 4500 7200 50  0001 C CNN
+	1    4500 7200
+	1    0    0    -1
+$EndComp
+$Comp
+L power:+3V3 #PWR0125
+U 1 1 5FA0862B
+P 4500 7050
+F 0 "#PWR0125" H 4500 6900 50  0001 C CNN
+F 1 "+3V3" H 4515 7223 50  0000 C CNN
+F 2 "" H 4500 7050 50  0001 C CNN
+F 3 "" H 4500 7050 50  0001 C CNN
+	1    4500 7050
+	1    0    0    -1
+$EndComp
+$Comp
+L power:GND #PWR0126
+U 1 1 5FA08635
+P 4500 7350
+F 0 "#PWR0126" H 4500 7100 50  0001 C CNN
+F 1 "GND" H 4505 7177 50  0000 C CNN
+F 2 "" H 4500 7350 50  0001 C CNN
+F 3 "" H 4500 7350 50  0001 C CNN
+	1    4500 7350
+	1    0    0    -1
+$EndComp
+$Comp
+L MCU_ST_STM32F0:STM32F051C6Tx U4
+U 1 1 5F72889D
+P 3450 4750
+F 0 "U4" H 2800 3100 50  0000 C CNN
+F 1 "STM32F041C6Tx" H 3050 3000 50  0000 C CNN
+F 2 "Housings_QFP:LQFP-48_7x7mm_Pitch0.5mm" H 2950 3250 50  0001 R CNN
+F 3 "http://www.st.com/st-web-ui/static/active/en/resource/technical/document/datasheet/DM00039193.pdf" H 3450 4750 50  0001 C CNN
+	1    3450 4750
+	1    0    0    -1
+$EndComp
+Wire Wire Line
+	2850 5450 2350 5450
+Wire Wire Line
+	2850 5550 2350 5550
+Text Label 2350 4750 0    50   ~ 0
+GPIO1
+Text Label 2350 5450 0    50   ~ 0
+GPIO2
+Text Label 2350 5550 0    50   ~ 0
+GPIO3
+Wire Wire Line
+	1400 800  1600 800
+$Comp
+L power:VDC #PWR0127
+U 1 1 5FA4D391
+P 1600 700
+F 0 "#PWR0127" H 1600 600 50  0001 C CNN
+F 1 "VDC" H 1615 873 50  0000 C CNN
+F 2 "" H 1600 700 50  0001 C CNN
+F 3 "" H 1600 700 50  0001 C CNN
+	1    1600 700
+	1    0    0    -1
+$EndComp
+Wire Wire Line
+	1600 700  1600 800
+Connection ~ 1600 800
+Wire Wire Line
+	1600 800  1750 800
+Wire Wire Line
+	4050 4650 4600 4650
+Wire Wire Line
+	4050 4750 4600 4750
+Wire Wire Line
+	4600 4850 4050 4850
+Wire Wire Line
+	4050 4950 4600 4950
+Wire Wire Line
+	4050 5250 4600 5250
+Wire Wire Line
+	4050 5350 4600 5350
+Wire Wire Line
+	2350 4650 2850 4650
+Text Label 4600 4650 2    50   ~ 0
+P1A
+Text Label 4600 4750 2    50   ~ 0
+P1B
+Text Label 4600 4850 2    50   ~ 0
+P2A
+Text Label 4600 4950 2    50   ~ 0
+P2B
+Text Label 4600 5250 2    50   ~ 0
+P3A
+Text Label 4600 5350 2    50   ~ 0
+P3B
+Text Label 2350 4650 0    50   ~ 0
+P4A
+Wire Wire Line
+	2350 4750 2850 4750
+Text Label 2350 5950 0    50   ~ 0
+P4B
+Wire Wire Line
+	2850 5950 2350 5950
+Wire Wire Line
+	2850 6050 2350 6050
+Text Label 2350 6050 0    50   ~ 0
+P5A
+Text Label 2350 6150 0    50   ~ 0
+P5B
+Wire Wire Line
+	2350 6150 2850 6150
+Wire Wire Line
+	2850 4850 2350 4850
+Wire Wire Line
+	2850 5650 2350 5650
+Wire Wire Line
+	2850 5750 2350 5750
+Text Label 2350 4850 0    50   ~ 0
+P1W
+Text Label 2350 5650 0    50   ~ 0
+P2W
+Text Label 2350 5750 0    50   ~ 0
+P3W
+Wire Wire Line
+	2850 5850 2350 5850
+Text Label 2350 5850 0    50   ~ 0
+P4W
+Wire Wire Line
+	4050 5450 4600 5450
+Text Label 4600 5450 2    50   ~ 0
+P5W
+$Comp
+L Connector:USB_B_Micro J4
+U 1 1 5BE2379A
+P 2200 2300
+F 0 "J4" H 2255 2767 50  0000 C CNN
+F 1 "USB_B_Micro" H 2255 2676 50  0000 C CNN
+F 2 "Connect:USB_Micro-B" H 2350 2250 50  0001 C CNN
+F 3 "~" H 2350 2250 50  0001 C CNN
+	1    2200 2300
+	1    0    0    -1
+$EndComp
+NoConn ~ 2100 2700
+NoConn ~ 4050 5050
+NoConn ~ 4050 5150
+NoConn ~ 4050 5550
+NoConn ~ 4050 5650
+NoConn ~ 2850 4950
+NoConn ~ 2850 5050
+NoConn ~ 2850 4250
+NoConn ~ 2850 3750
+NoConn ~ 2850 3850
 $EndSCHEMATC

Commit message: Final tweaks
Parts:
- added D26: YELLOW, LEDs:LED_0603, symbol Device:LED
- added R28: 470R, Resistors_SMD:R_0603, symbol Device:R
Connections:
- net GND: now also D26.1 (K)
- net HEARTBEAT: now reaches U4.40 (PB4)
- net HEARTBEAT: now also R28.1
- new net: D26.2 (A), R28.2
- no-connect marks 14 -> 13
Changed lines of the file:
@@
 Wire Wire Line
 	3450 6350 3450 6450
-Wire Wire Line
-	3350 3150 3450 3150
-Connection ~ 3450 3150
-Wire Wire Line
-	3450 3150 3550 3150
 Connection ~ 3550 3150
 Wire Wire Line
@@
 	1    0    0    -1
 $EndComp
-$Comp
-L MCU_ST_STM32F0:STM32F051C6Tx U4
-U 1 1 5F72889D
-P 3450 4750
-F 0 "U4" H 2800 3100 50  0000 C CNN
-F 1 "STM32F041C6Tx" H 3050 3000 50  0000 C CNN
-F 2 "Housings_QFP:LQFP-48_7x7mm_Pitch0.5mm" H 2950 3250 50  0001 R CNN
-F 3 "http://www.st.com/st-web-ui/static/active/en/resource/technical/document/datasheet/DM00039193.pdf" H 3450 4750 50  0001 C CNN
-	1    3450 4750
-	1    0    0    -1
-$EndComp
 Wire Wire Line
 	2850 5450 2350 5450
@@
 NoConn ~ 4050 5650
 NoConn ~ 2850 4950
-NoConn ~ 2850 5050
 NoConn ~ 2850 4250
 NoConn ~ 2850 3750
 NoConn ~ 2850 3850
+$Comp
+L Device:R R28
+U 1 1 5F87DE46
+P 1300 6800
+F 0 "R28" H 1370 6846 50  0000 L CNN
+F 1 "470R" H 1370 6755 50  0000 L CNN
+F 2 "Resistors_SMD:R_0603" V 1230 6800 50  0001 C CNN
+F 3 "~" H 1300 6800 50  0001 C CNN
+	1    1300 6800
+	1    0    0    -1
+$EndComp
+$Comp
+L power:GND #PWR01
+U 1 1 5F87DE50
+P 1300 7250
+F 0 "#PWR01" H 1300 7000 50  0001 C CNN
+F 1 "GND" H 1305 7077 50  0000 C CNN
+F 2 "" H 1300 7250 50  0001 C CNN
+F 3 "" H 1300 7250 50  0001 C CNN
+	1    1300 7250
+	1    0    0    -1
+$EndComp
+$Comp
+L Device:LED D26
+U 1 1 5F87DE5A
+P 1300 7100
+F 0 "D26" V 1338 6982 50  0000 R CNN
+F 1 "YELLOW" V 1247 6982 50  0000 R CNN
+F 2 "LEDs:LED_0603" H 1300 7100 50  0001 C CNN
+F 3 "~" H 1300 7100 50  0001 C CNN
+	1    1300 7100
+	0    -1   -1   0
+$EndComp
+Wire Wire Line
+	1300 6650 1300 6500
+Wire Wire Line
+	1300 6500 1900 6500
+Text Label 1900 6500 2    50   ~ 0
+HEARTBEAT
+Wire Wire Line
+	3450 3150 3550 3150
+Wire Wire Line
+	3350 3150 3450 3150
+Connection ~ 3450 3150
+$Comp
+L MCU_ST_STM32F0:STM32F051C6Tx U4
+U 1 1 5F72889D
+P 3450 4750
+F 0 "U4" H 2800 3100 50  0000 C CNN
+F 1 "STM32F041C6Tx" H 3050 3000 50  0000 C CNN
+F 2 "Housings_QFP:LQFP-48_7x7mm_Pitch0.5mm" H 2950 3250 50  0001 R CNN
+F 3 "http://www.st.com/st-web-ui/static/active/en/resource/technical/document/datasheet/DM00039193.pdf" H 3450 4750 50  0001 C CNN
+	1    3450 4750
+	1    0    0    -1
+$EndComp
+Wire Wire Line
+	2850 5050 2350 5050
+Text Label 2350 5050 0    50   ~ 0
+HEARTBEAT
 $EndSCHEMATC
