File: flowerpower/pot.sch (KiCad schematic (older format))
At the start: 13 parts, among them J7 Water sense, J8 Motor, U5 TB6559

Commit message: beginning layout
Parts:
- U5: footprint (none) -> flowerpower:16-hsop-fins
Changed lines of the file:
@@
 $Descr A4 11693 8268
 encoding utf-8
-Sheet 8 11
+Sheet 10 11
 Title ""
 Date ""
@@
 AR Path="/5FA12D65/5F85F211" Ref="D20"  Part="1"
 AR Path="/5FA1A820/5F85F211" Ref="D23"  Part="1"
-F 0 "D14" H 4793 2995 50  0000 C CNN
+F 0 "D20" H 4793 2995 50  0000 C CNN
 F 1 "BLUE" H 4793 3086 50  0000 C CNN
 F 2 "LEDs:LED_0603" H 4800 3250 50  0001 C CNN
@@
 AR Path="/5FA12D65/5F85FA74" Ref="R21"  Part="1"
 AR Path="/5FA1A820/5F85FA74" Ref="R25"  Part="1"
-F 0 "R13" V 4293 3250 50  0000 C CNN
+F 0 "R21" V 4293 3250 50  0000 C CNN
 F 1 "100R" V 4384 3250 50  0000 C CNN
 F 2 "Resistors_SMD:R_0603" V 4430 3250 50  0001 C CNN
@@
 AR Path="/5FA12D65/5F85FFAF" Ref="#PWR094"  Part="1"
 AR Path="/5FA1A820/5F85FFAF" Ref="#PWR0106"  Part="1"
-F 0 "#PWR0106" H 5050 3100 50  0001 C CNN
+F 0 "#PWR094" H 5050 3100 50  0001 C CNN
 F 1 "GND" H 5055 3177 50  0000 C CNN
 F 2 "" H 5050 3350 50  0001 C CNN
@@
 AR Path="/5FA12D65/5F86190F" Ref="R20"  Part="1"
 AR Path="/5FA1A820/5F86190F" Ref="R24"  Part="1"
-F 0 "R12" H 3520 2646 50  0000 L CNN
+F 0 "R20" H 3520 2646 50  0000 L CNN
 F 1 "2M2" H 3520 2555 50  0000 L CNN
 F 2 "Resistors_SMD:R_0603" V 3380 2600 50  0001 C CNN
@@
 AR Path="/5FA12D65/5F8625D7" Ref="#PWR091"  Part="1"
 AR Path="/5FA1A820/5F8625D7" Ref="#PWR0103"  Part="1"
-F 0 "#PWR0103" H 3450 2300 50  0001 C CNN
+F 0 "#PWR091" H 3450 2300 50  0001 C CNN
 F 1 "+3V3" H 3465 2623 50  0000 C CNN
 F 2 "" H 3450 2450 50  0001 C CNN
@@
 AR Path="/5FA12D65/5F862857" Ref="C23"  Part="1"
 AR Path="/5FA1A820/5F862857" Ref="C26"  Part="1"
-F 0 "C17" H 3565 3046 50  0000 L CNN
+F 0 "C23" H 3565 3046 50  0000 L CNN
 F 1 "10N" H 3565 2955 50  0000 L CNN
 F 2 "Capacitors_SMD:C_0603" H 3488 2850 50  0001 C CNN
@@
 AR Path="/5FA12D65/5F8629A0" Ref="#PWR093"  Part="1"
 AR Path="/5FA1A820/5F8629A0" Ref="#PWR0105"  Part="1"
-F 0 "#PWR0105" H 3450 2900 50  0001 C CNN
+F 0 "#PWR093" H 3450 2900 50  0001 C CNN
 F 1 "GND" H 3455 2977 50  0000 C CNN
 F 2 "" H 3450 3150 50  0001 C CNN
@@
 AR Path="/5FA12D65/5F862DB8" Ref="#PWR092"  Part="1"
 AR Path="/5FA1A820/5F862DB8" Ref="#PWR0104"  Part="1"
-F 0 "#PWR0104" H 3200 2900 50  0001 C CNN
+F 0 "#PWR092" H 3200 2900 50  0001 C CNN
 F 1 "GND" H 3205 2977 50  0000 C CNN
 F 2 "" H 3200 3150 50  0001 C CNN
@@
 AR Path="/5FA12D65/5F8631ED" Ref="J21"  Part="1"
 AR Path="/5FA1A820/5F8631ED" Ref="J23"  Part="1"
-F 0 "J17" H 2918 2625 50  0000 C CNN
+F 0 "J21" H 2918 2625 50  0000 C CNN
 F 1 "Water sense" H 2918 2716 50  0000 C CNN
 F 2 "Pin_Headers:Pin_Header_Straight_1x02" H 3000 2950 50  0001 C CNN
@@
 AR Path="/5FA12D65/5F863F1B" Ref="J22"  Part="1"
 AR Path="/5FA1A820/5F863F1B" Ref="J24"  Part="1"
-F 0 "J18" H 5130 4492 50  0000 L CNN
+F 0 "J22" H 5130 4492 50  0000 L CNN
 F 1 "Motor" H 5130 4401 50  0000 L CNN
 F 2 "Pin_Headers:Pin_Header_Straight_1x02" H 5050 4500 50  0001 C CNN
@@
 AR Path="/5FA12D65/5F867056" Ref="U8"  Part="1"
 AR Path="/5FA1A820/5F867056" Ref="U9"  Part="1"
-F 0 "U6" H 3950 4700 50  0000 L CNN
+F 0 "U8" H 3950 4700 50  0000 L CNN
 F 1 "TB6559" H 3850 4550 50  0000 L CNN
-F 2 "" H 3800 4200 50  0001 C CNN
+F 2 "flowerpower:16-hsop-fins" H 3800 4200 50  0001 C CNN
 F 3 "" H 3800 4200 50  0001 C CNN
 	1    4000 4550
@@
 AR Path="/5FA12D65/5F87101B" Ref="#PWR099"  Part="1"
 AR Path="/5FA1A820/5F87101B" Ref="#PWR0111"  Part="1"
-F 0 "#PWR0111" H 3850 5000 50  0001 C CNN
+F 0 "#PWR099" H 3850 5000 50  0001 C CNN
 F 1 "GND" H 3855 5077 50  0000 C CNN
 F 2 "" H 3850 5250 50  0001 C CNN
@@
 AR Path="/5FA12D65/5F8724E0" Ref="#PWR0100"  Part="1"
 AR Path="/5FA1A820/5F8724E0" Ref="#PWR0112"  Part="1"
-F 0 "#PWR0112" H 4350 5000 50  0001 C CNN
+F 0 "#PWR0100" H 4350 5000 50  0001 C CNN
 F 1 "GND" H 4355 5077 50  0000 C CNN
 F 2 "" H 4350 5250 50  0001 C CNN
@@
 AR Path="/5FA12D65/5F873D6D" Ref="#PWR096"  Part="1"
 AR Path="/5FA1A820/5F873D6D" Ref="#PWR0108"  Part="1"
-F 0 "#PWR0108" H 4150 3700 50  0001 C CNN
+F 0 "#PWR096" H 4150 3700 50  0001 C CNN
 F 1 "VDC" H 4165 3973 50  0000 C CNN
 F 2 "" H 4150 3800 50  0001 C CNN
@@
 AR Path="/5FA12D65/5F87F654" Ref="D22"  Part="1"
 AR Path="/5FA1A820/5F87F654" Ref="D25"  Part="1"
-F 0 "D16" V 2789 5082 50  0000 R CNN
+F 0 "D22" V 2789 5082 50  0000 R CNN
 F 1 "RED" V 2698 5082 50  0000 R CNN
 F 2 "LEDs:LED_0603" H 2750 5200 50  0001 C CNN
@@
 AR Path="/5FA12D65/5F87F65A" Ref="R23"  Part="1"
 AR Path="/5FA1A820/5F87F65A" Ref="R27"  Part="1"
-F 0 "R15" H 2680 4854 50  0000 R CNN
+F 0 "R23" H 2680 4854 50  0000 R CNN
 F 1 "680R" H 2680 4945 50  0000 R CNN
 F 2 "Resistors_SMD:R_0603" V 2680 4900 50  0001 C CNN
@@
 AR Path="/5FA12D65/5F87F660" Ref="#PWR0102"  Part="1"
 AR Path="/5FA1A820/5F87F660" Ref="#PWR0114"  Part="1"
-F 0 "#PWR0114" H 2750 5100 50  0001 C CNN
+F 0 "#PWR0102" H 2750 5100 50  0001 C CNN
 F 1 "GND" H 2755 5177 50  0000 C CNN
 F 2 "" H 2750 5350 50  0001 C CNN
@@
 AR Path="/5FA12D65/5F887B7F" Ref="#PWR0101"  Part="1"
 AR Path="/5FA1A820/5F887B7F" Ref="#PWR0113"  Part="1"
-F 0 "#PWR0113" H 2250 5100 50  0001 C CNN
+F 0 "#PWR0101" H 2250 5100 50  0001 C CNN
 F 1 "GND" H 2255 5177 50  0000 C CNN
 F 2 "" H 2250 5350 50  0001 C CNN
@@
 AR Path="/5FA12D65/5F883052" Ref="D21"  Part="1"
 AR Path="/5FA1A820/5F883052" Ref="D24"  Part="1"
-F 0 "D15" V 2289 5082 50  0000 R CNN
+F 0 "D21" V 2289 5082 50  0000 R CNN
 F 1 "GREEN" V 2198 5082 50  0000 R CNN
 F 2 "LEDs:LED_0603" H 2250 5200 50  0001 C CNN
@@
 AR Path="/5FA12D65/5F88C0E5" Ref="R22"  Part="1"
 AR Path="/5FA1A820/5F88C0E5" Ref="R26"  Part="1"
-F 0 "R14" H 2180 4854 50  0000 R CNN
+F 0 "R22" H 2180 4854 50  0000 R CNN
 F 1 "680R" H 2180 4945 50  0000 R CNN
 F 2 "Resistors_SMD:R_0603" V 2180 4900 50  0001 C CNN
@@
 AR Path="/5FA12D65/5F8927B4" Ref="#PWR097"  Part="1"
 AR Path="/5FA1A820/5F8927B4" Ref="#PWR0109"  Part="1"
-F 0 "#PWR0109" H 4750 3700 50  0001 C CNN
+F 0 "#PWR097" H 4750 3700 50  0001 C CNN
 F 1 "VDC" H 4765 3973 50  0000 C CNN
 F 2 "" H 4750 3800 50  0001 C CNN
@@
 AR Path="/5FA12D65/5F892BE3" Ref="C25"  Part="1"
 AR Path="/5FA1A820/5F892BE3" Ref="C28"  Part="1"
-F 0 "C19" H 4865 3996 50  0000 L CNN
+F 0 "C25" H 4865 3996 50  0000 L CNN
 F 1 "100N" H 4865 3905 50  0000 L CNN
 F 2 "Capacitors_SMD:C_0603" H 4788 3800 50  0001 C CNN
@@
 AR Path="/5FA12D65/5F893111" Ref="#PWR098"  Part="1"
 AR Path="/5FA1A820/5F893111" Ref="#PWR0110"  Part="1"
-F 0 "#PWR0110" H 4750 3850 50  0001 C CNN
+F 0 "#PWR098" H 4750 3850 50  0001 C CNN
 F 1 "GND" H 4755 3927 50  0000 C CNN
 F 2 "" H 4750 4100 50  0001 C CNN
@@
 AR Path="/5FA12D65/5F893789" Ref="C24"  Part="1"
 AR Path="/5FA1A820/5F893789" Ref="C27"  Part="1"
-F 0 "C18" H 3465 3696 50  0000 L CNN
+F 0 "C24" H 3465 3696 50  0000 L CNN
 F 1 "100N" H 3465 3605 50  0000 L CNN
 F 2 "Capacitors_SMD:C_0603" H 3388 3500 50  0001 C CNN
@@
 AR Path="/5FA12D65/5F89419E" Ref="#PWR095"  Part="1"
 AR Path="/5FA1A820/5F89419E" Ref="#PWR0107"  Part="1"
-F 0 "#PWR0107" H 3350 3550 50  0001 C CNN
+F 0 "#PWR095" H 3350 3550 50  0001 C CNN
 F 1 "GND" H 3355 3627 50  0000 C CNN
 F 2 "" H 3350 3800 50  0001 C CNN

Commit message: finish layout
Changed lines of the file:
@@
 $Descr A4 11693 8268
 encoding utf-8
-Sheet 10 11
+Sheet 2 11
 Title ""
 Date ""
@@
 AR Path="/5FA12D65/5F85F211" Ref="D20"  Part="1"
 AR Path="/5FA1A820/5F85F211" Ref="D23"  Part="1"
-F 0 "D20" H 4793 2995 50  0000 C CNN
+F 0 "D7" H 4793 2995 50  0000 C CNN
 F 1 "BLUE" H 4793 3086 50  0000 C CNN
 F 2 "LEDs:LED_0603" H 4800 3250 50  0001 C CNN
@@
 AR Path="/5FA12D65/5F85FA74" Ref="R21"  Part="1"
 AR Path="/5FA1A820/5F85FA74" Ref="R25"  Part="1"
-F 0 "R21" V 4293 3250 50  0000 C CNN
+F 0 "R7" V 4293 3250 50  0000 C CNN
 F 1 "100R" V 4384 3250 50  0000 C CNN
 F 2 "Resistors_SMD:R_0603" V 4430 3250 50  0001 C CNN
@@
 AR Path="/5FA12D65/5F86190F" Ref="R20"  Part="1"
 AR Path="/5FA1A820/5F86190F" Ref="R24"  Part="1"
-F 0 "R20" H 3520 2646 50  0000 L CNN
+F 0 "R6" H 3520 2646 50  0000 L CNN
 F 1 "2M2" H 3520 2555 50  0000 L CNN
 F 2 "Resistors_SMD:R_0603" V 3380 2600 50  0001 C CNN
@@
 AR Path="/5FA12D65/5F862857" Ref="C23"  Part="1"
 AR Path="/5FA1A820/5F862857" Ref="C26"  Part="1"
-F 0 "C23" H 3565 3046 50  0000 L CNN
+F 0 "C11" H 3565 3046 50  0000 L CNN
 F 1 "10N" H 3565 2955 50  0000 L CNN
 F 2 "Capacitors_SMD:C_0603" H 3488 2850 50  0001 C CNN
@@
 AR Path="/5FA12D65/5F8631ED" Ref="J21"  Part="1"
 AR Path="/5FA1A820/5F8631ED" Ref="J23"  Part="1"
-F 0 "J21" H 2918 2625 50  0000 C CNN
+F 0 "J7" H 2918 2625 50  0000 C CNN
 F 1 "Water sense" H 2918 2716 50  0000 C CNN
 F 2 "Pin_Headers:Pin_Header_Straight_1x02" H 3000 2950 50  0001 C CNN
@@
 AR Path="/5FA12D65/5F863F1B" Ref="J22"  Part="1"
 AR Path="/5FA1A820/5F863F1B" Ref="J24"  Part="1"
-F 0 "J22" H 5130 4492 50  0000 L CNN
+F 0 "J8" H 5130 4492 50  0000 L CNN
 F 1 "Motor" H 5130 4401 50  0000 L CNN
 F 2 "Pin_Headers:Pin_Header_Straight_1x02" H 5050 4500 50  0001 C CNN
@@
 AR Path="/5FA12D65/5F867056" Ref="U8"  Part="1"
 AR Path="/5FA1A820/5F867056" Ref="U9"  Part="1"
-F 0 "U8" H 3950 4700 50  0000 L CNN
+F 0 "U5" H 3950 4700 50  0000 L CNN
 F 1 "TB6559" H 3850 4550 50  0000 L CNN
 F 2 "flowerpower:16-hsop-fins" H 3800 4200 50  0001 C CNN
@@
 AR Path="/5FA12D65/5F87F654" Ref="D22"  Part="1"
 AR Path="/5FA1A820/5F87F654" Ref="D25"  Part="1"
-F 0 "D22" V 2789 5082 50  0000 R CNN
+F 0 "D9" V 2789 5082 50  0000 R CNN
 F 1 "RED" V 2698 5082 50  0000 R CNN
 F 2 "LEDs:LED_0603" H 2750 5200 50  0001 C CNN
@@
 AR Path="/5FA12D65/5F87F65A" Ref="R23"  Part="1"
 AR Path="/5FA1A820/5F87F65A" Ref="R27"  Part="1"
-F 0 "R23" H 2680 4854 50  0000 R CNN
+F 0 "R9" H 2680 4854 50  0000 R CNN
 F 1 "680R" H 2680 4945 50  0000 R CNN
 F 2 "Resistors_SMD:R_0603" V 2680 4900 50  0001 C CNN
@@
 AR Path="/5FA12D65/5F883052" Ref="D21"  Part="1"
 AR Path="/5FA1A820/5F883052" Ref="D24"  Part="1"
-F 0 "D21" V 2289 5082 50  0000 R CNN
+F 0 "D8" V 2289 5082 50  0000 R CNN
 F 1 "GREEN" V 2198 5082 50  0000 R CNN
 F 2 "LEDs:LED_0603" H 2250 5200 50  0001 C CNN
@@
 AR Path="/5FA12D65/5F88C0E5" Ref="R22"  Part="1"
 AR Path="/5FA1A820/5F88C0E5" Ref="R26"  Part="1"
-F 0 "R22" H 2180 4854 50  0000 R CNN
+F 0 "R8" H 2180 4854 50  0000 R CNN
 F 1 "680R" H 2180 4945 50  0000 R CNN
 F 2 "Resistors_SMD:R_0603" V 2180 4900 50  0001 C CNN
@@
 AR Path="/5FA12D65/5F892BE3" Ref="C25"  Part="1"
 AR Path="/5FA1A820/5F892BE3" Ref="C28"  Part="1"
-F 0 "C25" H 4865 3996 50  0000 L CNN
+F 0 "C13" H 4865 3996 50  0000 L CNN
 F 1 "100N" H 4865 3905 50  0000 L CNN
 F 2 "Capacitors_SMD:C_0603" H 4788 3800 50  0001 C CNN
@@
 AR Path="/5FA12D65/5F893789" Ref="C24"  Part="1"
 AR Path="/5FA1A820/5F893789" Ref="C27"  Part="1"
-F 0 "C24" H 3465 3696 50  0000 L CNN
+F 0 "C12" H 3465 3696 50  0000 L CNN
 F 1 "100N" H 3465 3605 50  0000 L CNN
 F 2 "Capacitors_SMD:C_0603" H 3388 3500 50  0001 C CNN

Commit message: Final tweaks
Changed lines of the file:
@@
 $Descr A4 11693 8268
 encoding utf-8
-Sheet 2 11
+Sheet 8 11
 Title ""
 Date ""
@@
 AR Path="/5FA12D65/5F85F211" Ref="D20"  Part="1"
 AR Path="/5FA1A820/5F85F211" Ref="D23"  Part="1"
-F 0 "D7" H 4793 2995 50  0000 C CNN
+F 0 "D23" H 4793 2995 50  0000 C CNN
 F 1 "BLUE" H 4793 3086 50  0000 C CNN
 F 2 "LEDs:LED_0603" H 4800 3250 50  0001 C CNN
@@
 AR Path="/5FA12D65/5F85FA74" Ref="R21"  Part="1"
 AR Path="/5FA1A820/5F85FA74" Ref="R25"  Part="1"
-F 0 "R7" V 4293 3250 50  0000 C CNN
+F 0 "R25" V 4293 3250 50  0000 C CNN
 F 1 "100R" V 4384 3250 50  0000 C CNN
 F 2 "Resistors_SMD:R_0603" V 4430 3250 50  0001 C CNN
@@
 AR Path="/5FA12D65/5F86190F" Ref="R20"  Part="1"
 AR Path="/5FA1A820/5F86190F" Ref="R24"  Part="1"
-F 0 "R6" H 3520 2646 50  0000 L CNN
+F 0 "R24" H 3520 2646 50  0000 L CNN
 F 1 "2M2" H 3520 2555 50  0000 L CNN
 F 2 "Resistors_SMD:R_0603" V 3380 2600 50  0001 C CNN
@@
 AR Path="/5FA12D65/5F862857" Ref="C23"  Part="1"
 AR Path="/5FA1A820/5F862857" Ref="C26"  Part="1"
-F 0 "C11" H 3565 3046 50  0000 L CNN
+F 0 "C26" H 3565 3046 50  0000 L CNN
 F 1 "10N" H 3565 2955 50  0000 L CNN
 F 2 "Capacitors_SMD:C_0603" H 3488 2850 50  0001 C CNN
@@
 AR Path="/5FA12D65/5F8631ED" Ref="J21"  Part="1"
 AR Path="/5FA1A820/5F8631ED" Ref="J23"  Part="1"
-F 0 "J7" H 2918 2625 50  0000 C CNN
+F 0 "J23" H 2918 2625 50  0000 C CNN
 F 1 "Water sense" H 2918 2716 50  0000 C CNN
 F 2 "Pin_Headers:Pin_Header_Straight_1x02" H 3000 2950 50  0001 C CNN
@@
 AR Path="/5FA12D65/5F863F1B" Ref="J22"  Part="1"
 AR Path="/5FA1A820/5F863F1B" Ref="J24"  Part="1"
-F 0 "J8" H 5130 4492 50  0000 L CNN
+F 0 "J24" H 5130 4492 50  0000 L CNN
 F 1 "Motor" H 5130 4401 50  0000 L CNN
 F 2 "Pin_Headers:Pin_Header_Straight_1x02" H 5050 4500 50  0001 C CNN
@@
 AR Path="/5FA12D65/5F867056" Ref="U8"  Part="1"
 AR Path="/5FA1A820/5F867056" Ref="U9"  Part="1"
-F 0 "U5" H 3950 4700 50  0000 L CNN
+F 0 "U9" H 3950 4700 50  0000 L CNN
 F 1 "TB6559" H 3850 4550 50  0000 L CNN
 F 2 "flowerpower:16-hsop-fins" H 3800 4200 50  0001 C CNN
@@
 AR Path="/5FA12D65/5F87F654" Ref="D22"  Part="1"
 AR Path="/5FA1A820/5F87F654" Ref="D25"  Part="1"
-F 0 "D9" V 2789 5082 50  0000 R CNN
+F 0 "D25" V 2789 5082 50  0000 R CNN
 F 1 "RED" V 2698 5082 50  0000 R CNN
 F 2 "LEDs:LED_0603" H 2750 5200 50  0001 C CNN
@@
 AR Path="/5FA12D65/5F87F65A" Ref="R23"  Part="1"
 AR Path="/5FA1A820/5F87F65A" Ref="R27"  Part="1"
-F 0 "R9" H 2680 4854 50  0000 R CNN
+F 0 "R27" H 2680 4854 50  0000 R CNN
 F 1 "680R" H 2680 4945 50  0000 R CNN
 F 2 "Resistors_SMD:R_0603" V 2680 4900 50  0001 C CNN
@@
 AR Path="/5FA12D65/5F883052" Ref="D21"  Part="1"
 AR Path="/5FA1A820/5F883052" Ref="D24"  Part="1"
-F 0 "D8" V 2289 5082 50  0000 R CNN
+F 0 "D24" V 2289 5082 50  0000 R CNN
 F 1 "GREEN" V 2198 5082 50  0000 R CNN
 F 2 "LEDs:LED_0603" H 2250 5200 50  0001 C CNN
@@
 AR Path="/5FA12D65/5F88C0E5" Ref="R22"  Part="1"
 AR Path="/5FA1A820/5F88C0E5" Ref="R26"  Part="1"
-F 0 "R8" H 2180 4854 50  0000 R CNN
+F 0 "R26" H 2180 4854 50  0000 R CNN
 F 1 "680R" H 2180 4945 50  0000 R CNN
 F 2 "Resistors_SMD:R_0603" V 2180 4900 50  0001 C CNN
@@
 AR Path="/5FA12D65/5F892BE3" Ref="C25"  Part="1"
 AR Path="/5FA1A820/5F892BE3" Ref="C28"  Part="1"
-F 0 "C13" H 4865 3996 50  0000 L CNN
+F 0 "C28" H 4865 3996 50  0000 L CNN
 F 1 "100N" H 4865 3905 50  0000 L CNN
 F 2 "Capacitors_SMD:C_0603" H 4788 3800 50  0001 C CNN
@@
 AR Path="/5FA12D65/5F893789" Ref="C24"  Part="1"
 AR Path="/5FA1A820/5F893789" Ref="C27"  Part="1"
-F 0 "C12" H 3465 3696 50  0000 L CNN
+F 0 "C27" H 3465 3696 50  0000 L CNN
 F 1 "100N" H 3465 3605 50  0000 L CNN
 F 2 "Capacitors_SMD:C_0603" H 3388 3500 50  0001 C CNN
